Commit message: [Error]:TF oscillation

File: turtle3/multiple_turtlebots_sim/urdf/turtlebot3_burger_one.gazebo.xacro (robot description, xacro)
@@ -3,8 +3,8 @@
   <xacro:arg name="laser_visual" default="true"/>
   <xacro:arg name="imu_visual"   default="false"/>
-  <gazebo reference="base_link">
+  <gazebo reference="tb3_0/base_link">
     <material>Gazebo/DarkGrey</material>
   </gazebo>
-  <gazebo reference="wheel_left_link">
+  <gazebo reference="tb3_0/wheel_left_link">
     <mu1>0.1</mu1>
     <mu2>0.1</mu2>
@@ -16,5 +16,5 @@
     <material>Gazebo/FlatBlack</material>
   </gazebo>
-  <gazebo reference="wheel_right_link">
+  <gazebo reference="tb3_0/wheel_right_link">
     <mu1>0.1</mu1>
     <mu2>0.1</mu2>
@@ -26,5 +26,5 @@
     <material>Gazebo/FlatBlack</material>
   </gazebo>
-  <gazebo reference="caster_back_link">
+  <gazebo reference="tb3_0/caster_back_link">
     <mu1>0.1</mu1>
     <mu2>0.1</mu2>
@@ -35,5 +35,5 @@
     <material>Gazebo/FlatBlack</material>
   </gazebo>
-  <gazebo reference="imu_link">
+  <gazebo reference="tb3_0/imu_link">
     <sensor type="imu" name="imu">
       <always_on>true</always_on>
@@ -92,5 +92,5 @@
     </plugin>
   </gazebo>
-  <gazebo reference="base_scan">
+  <gazebo reference="tb3_0/base_scan">
     <material>Gazebo/FlatBlack</material>
     <sensor type="ray" name="lds_lfcd_sensor">

File: turtle3/multiple_turtlebots_sim/urdf/turtlebot3_burger_one.urdf.xacro (robot description, xacro)
@@ -3,11 +3,11 @@
   <xacro:include filename="$(find turtlebot3_description)/urdf/common_properties.xacro"/>
   <xacro:include filename="$(find multiple_turtlebots_sim)/urdf/turtlebot3_burger.gazebo.xacro"/>
-  <link name="base_footprint"/>
-  <joint name="base_joint" type="fixed">
-    <parent link="base_footprint"/>
-    <child link="base_link"/>
+  <link name="tb3_0/base_footprint"/>
+  <joint name="tb3_0/base_joint" type="fixed">
+    <parent link="tb3_0/base_footprint"/>
+    <child link="tb3_0/base_link"/>
     <origin xyz="0.0 0.0 0.010" rpy="0 0 0"/>
   </joint>
-  <link name="base_link">
+  <link name="tb3_0/base_link">
     <visual>
       <origin xyz="-0.032 0 0.0" rpy="0 0 0"/>
@@ -31,11 +31,11 @@
     </inertial>
   </link>
-  <joint name="wheel_left_joint" type="continuous">
-    <parent link="base_link"/>
-    <child link="wheel_left_link"/>
+  <joint name="tb3_0/wheel_left_joint" type="continuous">
+    <parent link="tb3_0/base_link"/>
+    <child link="tb3_0/wheel_left_link"/>
     <origin xyz="0.0 0.08 0.023" rpy="-1.57 0 0"/>
     <axis xyz="0 0 1"/>
   </joint>
-  <link name="wheel_left_link">
+  <link name="tb3_0/wheel_left_link">
     <visual>
       <origin xyz="0 0 0" rpy="1.57 0 0"/>
@@ -59,11 +59,11 @@
       </inertial>
   </link>
-  <joint name="wheel_right_joint" type="continuous">
-    <parent link="base_link"/>
-    <child link="wheel_right_link"/>
+  <joint name="tb3_0/wheel_right_joint" type="continuous">
+    <parent link="tb3_0/base_link"/>
+    <child link="tb3_0/wheel_right_link"/>
     <origin xyz="0.0 -0.080 0.023" rpy="-1.57 0 0"/>
     <axis xyz="0 0 1"/>
   </joint>
-  <link name="wheel_right_link">
+  <link name="tb3_0/wheel_right_link">
     <visual>
       <origin xyz="0 0 0" rpy="1.57 0 0"/>
@@ -87,10 +87,10 @@
       </inertial>
   </link>
-  <joint name="caster_back_joint" type="fixed">
-    <parent link="base_link"/>
-    <child link="caster_back_link"/>
+  <joint name="tb3_0/caster_back_joint" type="fixed">
+    <parent link="tb3_0/base_link"/>
+    <child link="tb3_0/caster_back_link"/>
     <origin xyz="-0.081 0 -0.004" rpy="-1.57 0 0"/>
   </joint>
-  <link name="caster_back_link">
+  <link name="tb3_0/caster_back_link">
     <collision>
       <origin xyz="0 0.001 0" rpy="0 0 0"/>
@@ -107,16 +107,16 @@
     </inertial>
   </link>
-  <joint name="imu_joint" type="fixed">
-    <parent link="base_link"/>
-    <child link="imu_link"/>
+  <joint name="tb3_0/imu_joint" type="fixed">
+    <parent link="tb3_0/base_link"/>
+    <child link="tb3_0/imu_link"/>
     <origin xyz="-0.032 0 0.068" rpy="0 0 0"/>
   </joint>
-  <link name="imu_link"/>
+  <link name="tb3_0/imu_link"/>
   <joint name="scan_joint" type="fixed">
-    <parent link="base_link"/>
-    <child link="base_scan"/>
+    <parent link="tb3_0/base_link"/>
+    <child link="tb3_0/base_scan"/>
     <origin xyz="-0.032 0 0.172" rpy="0 0 0"/>
   </joint>
-  <link name="base_scan">
+  <link name="tb3_0/base_scan">
     <visual>
       <origin xyz="0 0 0.0" rpy="0 0 0"/>

File: turtle3/multiple_turtlebots_sim/urdf/turtlebot3_burger_two.gazebo.xacro (robot description, xacro)
@@ -3,8 +3,8 @@
   <xacro:arg name="laser_visual" default="true"/>
   <xacro:arg name="imu_visual"   default="false"/>
-  <gazebo reference="tb3_1/base_link">
+  <gazebo reference="base_link">
     <material>Gazebo/DarkGrey</material>
   </gazebo>
-  <gazebo reference="tb3_1/wheel_left_link">
+  <gazebo reference="wheel_left_link">
     <mu1>0.1</mu1>
     <mu2>0.1</mu2>
@@ -16,5 +16,5 @@
     <material>Gazebo/FlatBlack</material>
   </gazebo>
-  <gazebo reference="tb3_1/wheel_right_link">
+  <gazebo reference="wheel_right_link">
     <mu1>0.1</mu1>
     <mu2>0.1</mu2>
@@ -26,5 +26,5 @@
     <material>Gazebo/FlatBlack</material>
   </gazebo>
-  <gazebo reference="tb3_1/caster_back_link">
+  <gazebo reference="caster_back_link">
     <mu1>0.1</mu1>
     <mu2>0.1</mu2>
@@ -35,5 +35,5 @@
     <material>Gazebo/FlatBlack</material>
   </gazebo>
-  <gazebo reference="tb3_1/imu_link">
+  <gazebo reference="imu_link">
     <sensor type="imu" name="imu">
       <always_on>true</always_on>
@@ -92,5 +92,5 @@
     </plugin>
   </gazebo>
-  <gazebo reference="tb3_1/base_scan">
+  <gazebo reference="base_scan">
     <material>Gazebo/FlatBlack</material>
     <sensor type="ray" name="lds_lfcd_sensor">
